File: PCB/PCBruler.kicad_pcb (KiCad board)
At the start: 2 copper layers, 156 x 26 mm, 15 parts, among them Q1/T1 TO-92, Q2/T2 TO-220-3_Vertical

Commit message: draft of the back
Parts:
- added J1: USB_C_Receptacle_HRO_TYPE-C-31-M-12, Connector_USB:USB_C_Receptacle_HRO_TYPE-C-31-M-12, B.Cu at (64.8, 4.00)
- added Q3/T3: SOT-323_SC-70, Package_TO_SOT_SMD:SOT-323_SC-70, F.Cu at (109.8, 23.5)
- added REF**: C_0603_1608Metric, Capacitor_SMD:C_0603_1608Metric, B.Cu at (86.8, 15.5)
- added REF**: C_0201_0603Metric, Capacitor_SMD:C_0201_0603Metric, B.Cu at (86.8, 18.5)
- added REF**: C_0805_2012Metric, Capacitor_SMD:C_0805_2012Metric, B.Cu at (86.8, 13.5)
- added REF**: L_1206_3216Metric, Inductor_SMD:L_1206_3216Metric, B.Cu at (86.8, 11.0)
- added REF**: C_0402_1005Metric, Capacitor_SMD:C_0402_1005Metric, B.Cu at (86.8, 17.2)
- added REF**: C_1210_3225Metric, Capacitor_SMD:C_1210_3225Metric, B.Cu at (86.8, 8.00)
- added U1: SOIC-8_5.3x5.3mm_P1.27mm, Package_SO:SOIC-8_5.3x5.3mm_P1.27mm, B.Cu at (69.2, 23.0)
- added U2: SOIC-16_3.9x9.9mm_P1.27mm, Package_SO:SOIC-16_3.9x9.9mm_P1.27mm, B.Cu at (76.8, 11.2)
- added U4: QFN-32-1EP_4x4mm_P0.4mm_EP2.65x2.65mm, Package_DFN_QFN:QFN-32-1EP_4x4mm_P0.4mm_EP2.65x2.65mm, B.Cu at (64.8, 13.7)
- added U5: LQFP-64-1EP_10x10mm_P0.5mm_EP5x5mm, Package_QFP:LQFP-64-1EP_10x10mm_P0.5mm_EP5x5mm, B.Cu at (51.2, 8.75)
- added U6: TO-252-2, Package_TO_SOT_SMD:TO-252-2, B.Cu at (38.7, 8.16)
- added U7: SOT-223, Package_TO_SOT_SMD:SOT-223, B.Cu at (27.0, 5.75)
- added U8: TFBGA-64_5x5mm_Layout8x8_P0.5mm, Package_BGA:TFBGA-64_5x5mm_Layout8x8_P0.5mm, B.Cu at (29.0, 16.5)
- added U9: LED_WS2812B_PLCC4_5.0x5.0mm_P3.2mm, LED_SMD:LED_WS2812B_PLCC4_5.0x5.0mm_P3.2mm, B.Cu at (52.8, 23.0)
- added U9: ESP32-WROOM-32E, RF_Module:ESP32-WROOM-32E, B.Cu at (9.75, 6.01)
- moved D7 14.9 mm to (148.6, 23.4), turned to 0 degrees
- moved R6 8.05 mm to (152.2, 23.4), turned to 180 degrees
- moved Q1/T1 2.19 mm to (92.5, 13.4)
- moved E$50 1.75 mm to (119.2, 17.2)
- moved E$54 1.75 mm to (105.8, 17.2)
- moved E$59 1.75 mm to (112.2, 17.2)
Other:
- board text added: "1 kΩ = 1000 Ω | 1 µF = 1000 nF = 1 000 000 pF"
- board text added: "DPAK"
- board text added: "Je rychlý a zvládne i WiFi a Bluethooth"
- board text added: "RFID Detektor"
- board text added: "R_ser = R1 + R2 | R_par = (R1 * R2) / (R1 + R2) C_par = C1 + C2 | C_ser = (C1 * C2) / (C1 + C2)"
- board text added: "SMD R/C/L"
- board text added: "Tabulky"
- board text added: "Toto je pouzro pro mikrokontrolér ESP32"
- board text added: "U = R * I | P = U * I | Q = C * U"
- board text added: "tau = R * C | fc = 1 / (2 * pi * R * C)"
- board text removed: "1 µF = 1000 nF = 1 000 000 pF | 1 kΩ = 1000 Ω"
- board text removed: "Transformátor"

Commit message: finished the back and graphics
Other:
- board text added: "Jméno"

Commit message: finishing touches on the PCB
Other:
- board text added: "by Tk"
